File: hardware/mshv2/esp32.kicad_sch (KiCad schematic)
At the start: 0 parts

Commit message: feat: Implement KiCad schematic Parts 0-3 and update dashboard I/O to 2 LEDs
KiCad Schematic Implementation:
- Part 0: Created hierarchical sheet structure (power, ESP32, sensors, I/O)
- Part 1: Implemented power supply sheet with dual power OR-ing diodes
- Part 2: Completed ESP32 Core sheet with GPIO assignments and USB-C
- Part 3: Built current sensing sheet with 5-channel op-amp conditioning

Documentation Updates (Breaking Change):
- Reduced dashboard I/O from 3 LEDs to 2 LEDs (GPIO11, GPIO15)
- Kept 3 switch inputs (GPIO16, GPIO17, GPIO23)
- GPIO14 not available on ESP32-C6-WROOM-1 module (used internally)
- Updated Hardware.md, Requirements.md, README.md, KICAD_SCHEMATIC_GUIDE.md
- J_IO connector reduced from 10-pin to 9-pin
- BOM updated: 2× MOSFETs (was 3×), cost reduced to $35.85 (was $36.00)

Markdown Linting:
- Fixed all markdown lint warnings in LICENSE and Hardware.md
- Converted bold license headings to proper H2/H3 headings
- Added blank lines around all lists
- Wrapped bare URLs in angle brackets
- Escaped glob patterns in file listings

BREAKING CHANGE: Dashboard I/O reduced to 2 LED outputs (GPIO11, GPIO15)
due to GPIO14 being unavailable on ESP32-C6-WROOM-1 module. GPIO14 is used
internally for flash memory and not broken out to module pins.

🤖 Generated with [Claude Code](https://claude.com/claude-code)

Co-Authored-By: Claude Sonnet 4.5 <noreply@anthropic.com>
Parts:
- added C_EN1, C_RGB: 0.1uF, Capacitor_SMD:C_0201_0603Metric, symbol Device:C
- added C_USB_IN: 10uF, Capacitor_SMD:C_0201_0603Metric, symbol Device:C
- added C_USB_SHIELD: 100nF, Capacitor_SMD:C_0201_0603Metric, symbol Device:C
- added D_PWR: Green LED, LED_SMD:LED_0603_1608Metric, symbol Device:LED
- added D_RGB: WS2812B, LED_SMD:LED_WS2812B_PLCC4_5.0x5.0mm_P3.2mm, symbol LED:WS2812B
- added D_USB: B5819W, Diode_SMD:D_0201_0603Metric, symbol Device:D_Schottky
- added J_USB: USB_C_Receptacle_USB2.0_16P, Connector_USB:USB_C_Receptacle_GCT_USB4105-xx-A_16P_TopMnt_Horizontal, symbol Connector:USB_C_Receptacle_USB2.0_16P
- added R_BOOT, R_EN: 10k, Resistor_SMD:R_0201_0603Metric, symbol Device:R
- added R_CC1, R_CC2: 5.1k, Resistor_SMD:R_0201_0603Metric, symbol Device:R
- added R_PWR: 1k, Resistor_SMD:R_0201_0603Metric, symbol Device:R
- added R_RBG: 330, Resistor_SMD:R_0201_0603Metric, symbol Device:R
- added SW_BOOT, SW_RESET: SW_Push, Button_Switch_THT:SW_Tactile_Straight_KSA0Axx1LFTR, symbol Switch:SW_Push
- added U3: AMS1117-3.3, Package_TO_SOT_SMD:SOT-223-3_TabPin2, symbol Regulator_Linear:AMS1117-3.3
- added U4: ESP32-C6-WROOM-1-N8, PCM_Espressif:ESP32-C6-WROOM-1, symbol PCM_Espressif:ESP32-C6-WROOM-1
- added U_ESD: USBLC6-2SC6, Package_TO_SOT_SMD:SOT-23-6, symbol Power_Protection:USBLC6-2SC6
Connections:
- new net: R_BOOT.1, U4.15 (GPIO9)
- new net: R_EN.2, U4.3 (EN/CHIP_PU)
- new net: J_USB.A5 (CC1), R_CC2.1
- new net: C_USB_IN.1, J_USB.A4 (VBUS), J_USB.A9 (VBUS), J_USB.B4 (VBUS), J_USB.B9 (VBUS), U3.3 (VI), U_ESD.4 (I/O2)
- new net: D_PWR.2 (A), R_PWR.1
- new net: D_RGB.4 (DIN), R_RBG.2
- new net: J_USB.A7 (D-), J_USB.B7 (D-), U_ESD.1 (I/O1)
- new net: J_USB.A6 (D+), J_USB.B6 (D+), U_ESD.3 (I/O2)
- new net: D_USB.2 (A), U3.2 (VO)
- new net: J_USB.B5 (CC2), R_CC1.2
- new net: C_USB_SHIELD.1, J_USB.S1 (SHIELD)
- new net +3.3V: C_EN1.1, R_EN.1, SW_RESET.2
- new net +3V3: C_RGB.2, D_RGB.1 (VDD), D_USB.1 (K), R_BOOT.2, R_PWR.2, SW_BOOT.1, U4.2 (3V3)
- new net 1WIRE_DATA: U4.11 (GPIO10)
- new net ADC_CH0: U4.8 (GPIO0/ADC1_CH0/XTAL_32K_P)
- new net ADC_CH1: U4.9 (GPIO1/ADC1_CH1/XTAL_32K_N)
- new net ADC_CH2: U4.27 (GPIO2/ADC1_CH2)
- new net ADC_CH3: U4.26 (GPIO3/ADC1_CH3)
- new net ADC_CH4: U4.4 (MTMS/GPIO4/ADC1_CH4)
- new net GND: C_EN1.2, C_RGB.1, C_USB_IN.2, C_USB_SHIELD.2, D_PWR.1 (K), D_RGB.3 (VSS), J_USB.A1 (GND), J_USB.A12 (GND), J_USB.B1 (GND), J_USB.B12 (GND), R_CC1.1, R_CC2.2, SW_BOOT.2, SW_RESET.1, U3.1 (GND), U4.1 (GND), U4.28 (GND), U4.29 (GND), U_ESD.2 (GND)
- new net I2C_SCL: U4.7 (MTDO/GPIO7)
- new net I2C_SDA: U4.6 (MTCK/GPIO6/ADC1_CH6)
- new net LED1_OUT: U4.12 (GPIO11)
- new net LED2_OUT: U4.23 (GPIO15)
- new net PIEZO: U4.5 (MTDI/GPIO5/ADC1_CH5)
- new net RGB_LED: R_RBG.1, U4.10 (GPIO8)
- new net SPI_CS_TC1: U4.18 (GPIO20)
- new net SPI_CS_TC2: U4.19 (GPIO21)
- new net SPI_CS_TC3: U4.20 (GPIO22)
- new net SPI_MISO: U4.16 (GPIO18)
- new net SPI_SCK: U4.17 (GPIO19)
- new net SWITCH1_IN: U4.25 (U0TXD/GPIO16)
- new net SWITCH2_IN: U4.24 (U0RXD/GPIO17)
- new net SWITCH3_IN: U4.21 (GPIO23)
- new net USB_D+: U4.14 (GPIO13/USB_D+), U_ESD.6 (I/O1)
- new net USB_D-: U4.13 (GPIO12/USB_D-), U_ESD.5 (VBUS)
- no-connect marks 0 -> 2
Other:
- company: (none) -> Don McGarry
