File: hardware/mshv2/mshv2.kicad_sch (KiCad schematic)
At the start: 63 parts, among them J1 12V_INPUT, J2 CLAMP_1, J3 CLAMP_2, J4 CLAMP_3, J5 CLAMP_4, J6 CLAMP_5, U1 LM2596S-3.3, U2 MCP6004, U3 AMS1117-3.3, U4 ESP32-C6-WROOM-1-N8, U5 MCP6004

Commit message: feat: Implement KiCad schematic Parts 0-3 and update dashboard I/O to 2 LEDs
KiCad Schematic Implementation:
- Part 0: Created hierarchical sheet structure (power, ESP32, sensors, I/O)
- Part 1: Implemented power supply sheet with dual power OR-ing diodes
- Part 2: Completed ESP32 Core sheet with GPIO assignments and USB-C
- Part 3: Built current sensing sheet with 5-channel op-amp conditioning

Documentation Updates (Breaking Change):
- Reduced dashboard I/O from 3 LEDs to 2 LEDs (GPIO11, GPIO15)
- Kept 3 switch inputs (GPIO16, GPIO17, GPIO23)
- GPIO14 not available on ESP32-C6-WROOM-1 module (used internally)
- Updated Hardware.md, Requirements.md, README.md, KICAD_SCHEMATIC_GUIDE.md
- J_IO connector reduced from 10-pin to 9-pin
- BOM updated: 2× MOSFETs (was 3×), cost reduced to $35.85 (was $36.00)

Markdown Linting:
- Fixed all markdown lint warnings in LICENSE and Hardware.md
- Converted bold license headings to proper H2/H3 headings
- Added blank lines around all lists
- Wrapped bare URLs in angle brackets
- Escaped glob patterns in file listings

BREAKING CHANGE: Dashboard I/O reduced to 2 LED outputs (GPIO11, GPIO15)
due to GPIO14 being unavailable on ESP32-C6-WROOM-1 module. GPIO14 is used
internally for flash memory and not broken out to module pins.

🤖 Generated with [Claude Code](https://claude.com/claude-code)

Co-Authored-By: Claude Sonnet 4.5 <noreply@anthropic.com>
Parts:
- removed C1: 100uF/25V, Capacitor_SMD:C_0201_0603Metric, symbol Device:C_Polarized
- removed C2: 100uF/10V, Capacitor_SMD:C_0201_0603Metric, symbol Device:C_Polarized
- removed C3, C_USB_IN1: 10uF, Capacitor_SMD:C_0201_0603Metric, symbol Device:C
- removed C4, C_EN1, C_FILT_1, C_FILT_2, C_FILT_3, C_FILT_4, C_FILT_5, C_FILT_E_1, C_FILT_E_2, C_RGB1: 0.1uF, Capacitor_SMD:C_0201_0603Metric, symbol Device:C
- removed C_USB_SHIELD1: 100nF, Capacitor_SMD:C_0201_0603Metric, symbol Device:C
- removed D1: MBRS340, Diode_SMD:D_SMC, symbol Diode:MBRS340
- removed D_BUCK1, D_USB1: B5819W, Diode_SMD:D_0201_0603Metric, symbol Device:D_Schottky
- removed D_PWR1, D_STATUS1: Green LED, LED_SMD:LED_0603_1608Metric, symbol Device:LED
- removed D_RGB1: WS2812B, LED_SMD:LED_WS2812B_PLCC4_5.0x5.0mm_P3.2mm, symbol LED:WS2812B
- removed J1: 12V_INPUT, TerminalBlock:TerminalBlock_MaiXu_MX126-5.0-02P_1x02_P5.00mm, symbol Connector:Screw_Terminal_01x02
- removed J2: CLAMP_1, TerminalBlock:TerminalBlock_MaiXu_MX126-5.0-02P_1x02_P5.00mm, symbol Connector:Screw_Terminal_01x02
- removed J3: CLAMP_2, TerminalBlock:TerminalBlock_MaiXu_MX126-5.0-02P_1x02_P5.00mm, symbol Connector:Screw_Terminal_01x02
- removed J4: CLAMP_3, TerminalBlock:TerminalBlock_MaiXu_MX126-5.0-02P_1x02_P5.00mm, symbol Connector:Screw_Terminal_01x02
- removed J5: CLAMP_4, TerminalBlock:TerminalBlock_MaiXu_MX126-5.0-02P_1x02_P5.00mm, symbol Connector:Screw_Terminal_01x02
- removed J6: CLAMP_5, TerminalBlock:TerminalBlock_MaiXu_MX126-5.0-02P_1x02_P5.00mm, symbol Connector:Screw_Terminal_01x02
- removed J_USB1: USB_C_Receptacle_USB2.0_16P, Connector_USB:USB_C_Receptacle_GCT_USB4105-xx-A_16P_TopMnt_Horizontal, symbol Connector:USB_C_Receptacle_USB2.0_16P
- removed R_BOOT1, R_DIV1_1, R_DIV1_2, R_DIV1_3, R_DIV1_4, R_DIV1_5, R_EN1: 10k, Resistor_SMD:R_0201_0603Metric, symbol Device:R
- removed R_CC1, R_CC2: 5.1k, Resistor_SMD:R_0201_0603Metric, symbol Device:R
- removed R_DIV2_1, R_DIV2_2, R_DIV2_3, R_DIV2_4, R_DIV2_5: 20k, Resistor_SMD:R_0201_0603Metric, symbol Device:R
- removed R_FILT_1, R_FILT_2, R_FILT_3, R_FILT_4, R_FILT_5, R_PWR1, R_SER_1, R_SER_2, R_SER_3, R_SER_4, R_SER_5: 1k, Resistor_SMD:R_0201_0603Metric, symbol Device:R
- removed R_RBG1, R_STATUS1: 330, Resistor_SMD:R_0201_0603Metric, symbol Device:R
- removed SW_BOOT1, SW_RESET1: SW_Push, Button_Switch_THT:SW_Tactile_Straight_KSA0Axx1LFTR, symbol Switch:SW_Push
- removed U1: LM2596S-3.3, Package_TO_SOT_SMD:TO-263-5_TabPin3, symbol Regulator_Switching:LM2596S-3.3
- removed U2, U5: MCP6004, Package_SO:SOIC-14_3.9x8.7mm_P1.27mm, symbol Amplifier_Operational:MCP6004
- removed U3: AMS1117-3.3, Package_TO_SOT_SMD:SOT-223-3_TabPin2, symbol Regulator_Linear:AMS1117-3.3
- removed U4: ESP32-C6-WROOM-1-N8, PCM_Espressif:ESP32-C6-WROOM-1, symbol PCM_Espressif:ESP32-C6-WROOM-1
- removed U_ESD1: USBLC6-2SC6, Package_TO_SOT_SMD:SOT-23-6, symbol Power_Protection:USBLC6-2SC6
Other:
- sheet ESP32 ports: added +3V3, 1WIRE_DATA, ADC_CH0, ADC_CH1, ADC_CH2, ADC_CH3, ADC_CH4, GND, I2C_SCL, I2C_SDA, LED1_OUT, LED2_OUT, PIEZO, SPI_CS_TC1, SPI_CS_TC2, SPI_CS_TC3, SPI_MISO, SPI_SCK, SWITCH1_IN, SWITCH2_IN, SWITCH3_IN; removed none
- sheet Power Supply ports: added +12V, +3V3, GND; removed none
