File: hardware/mshv2/power.kicad_sch (KiCad schematic)
At the start: 0 parts

Commit message: feat: Implement KiCad schematic Parts 0-3 and update dashboard I/O to 2 LEDs
KiCad Schematic Implementation:
- Part 0: Created hierarchical sheet structure (power, ESP32, sensors, I/O)
- Part 1: Implemented power supply sheet with dual power OR-ing diodes
- Part 2: Completed ESP32 Core sheet with GPIO assignments and USB-C
- Part 3: Built current sensing sheet with 5-channel op-amp conditioning

Documentation Updates (Breaking Change):
- Reduced dashboard I/O from 3 LEDs to 2 LEDs (GPIO11, GPIO15)
- Kept 3 switch inputs (GPIO16, GPIO17, GPIO23)
- GPIO14 not available on ESP32-C6-WROOM-1 module (used internally)
- Updated Hardware.md, Requirements.md, README.md, KICAD_SCHEMATIC_GUIDE.md
- J_IO connector reduced from 10-pin to 9-pin
- BOM updated: 2× MOSFETs (was 3×), cost reduced to $35.85 (was $36.00)

Markdown Linting:
- Fixed all markdown lint warnings in LICENSE and Hardware.md
- Converted bold license headings to proper H2/H3 headings
- Added blank lines around all lists
- Wrapped bare URLs in angle brackets
- Escaped glob patterns in file listings

BREAKING CHANGE: Dashboard I/O reduced to 2 LED outputs (GPIO11, GPIO15)
due to GPIO14 being unavailable on ESP32-C6-WROOM-1 module. GPIO14 is used
internally for flash memory and not broken out to module pins.

🤖 Generated with [Claude Code](https://claude.com/claude-code)

Co-Authored-By: Claude Sonnet 4.5 <noreply@anthropic.com>
Parts:
- added C1: 100uF/25V, Capacitor_SMD:C_0201_0603Metric, symbol Device:C_Polarized
- added C2: 100uF/10V, Capacitor_SMD:C_0201_0603Metric, symbol Device:C_Polarized
- added C3: 10uF, Capacitor_SMD:C_0201_0603Metric, symbol Device:C
- added C4: 0.1uF, Capacitor_SMD:C_0201_0603Metric, symbol Device:C
- added D1: MBRS340, Diode_SMD:D_SMC, symbol Diode:MBRS340
- added D_BUCK: B5819W, Diode_SMD:D_0201_0603Metric, symbol Device:D_Schottky
- added U1: LM2596S-3.3, Package_TO_SOT_SMD:TO-263-5_TabPin3, symbol Regulator_Switching:LM2596S-3.3
Connections:
- new net: C2.1, C3.1, D_BUCK.2 (A), U1.2 (OUT), U1.4 (FB)
- new net: C1.1, D1.1 (K), U1.1 (VIN), U1.5 (~{ON}/OFF)
- new net +12V: D1.2 (A)
- new net +3V3: C4.1, D_BUCK.1 (K)
- new net GND: C1.2, C2.2, C3.2, C4.2, U1.3 (GND)
Other:
- company: (none) -> Don McGarry
