File: hardware/mshv2/sensors_current.kicad_sch (KiCad schematic)
At the start: 0 parts

Commit message: feat: Implement KiCad schematic Parts 0-3 and update dashboard I/O to 2 LEDs
KiCad Schematic Implementation:
- Part 0: Created hierarchical sheet structure (power, ESP32, sensors, I/O)
- Part 1: Implemented power supply sheet with dual power OR-ing diodes
- Part 2: Completed ESP32 Core sheet with GPIO assignments and USB-C
- Part 3: Built current sensing sheet with 5-channel op-amp conditioning

Documentation Updates (Breaking Change):
- Reduced dashboard I/O from 3 LEDs to 2 LEDs (GPIO11, GPIO15)
- Kept 3 switch inputs (GPIO16, GPIO17, GPIO23)
- GPIO14 not available on ESP32-C6-WROOM-1 module (used internally)
- Updated Hardware.md, Requirements.md, README.md, KICAD_SCHEMATIC_GUIDE.md
- J_IO connector reduced from 10-pin to 9-pin
- BOM updated: 2× MOSFETs (was 3×), cost reduced to $35.85 (was $36.00)

Markdown Linting:
- Fixed all markdown lint warnings in LICENSE and Hardware.md
- Converted bold license headings to proper H2/H3 headings
- Added blank lines around all lists
- Wrapped bare URLs in angle brackets
- Escaped glob patterns in file listings

BREAKING CHANGE: Dashboard I/O reduced to 2 LED outputs (GPIO11, GPIO15)
due to GPIO14 being unavailable on ESP32-C6-WROOM-1 module. GPIO14 is used
internally for flash memory and not broken out to module pins.

🤖 Generated with [Claude Code](https://claude.com/claude-code)

Co-Authored-By: Claude Sonnet 4.5 <noreply@anthropic.com>
Parts:
- added C_FILT_1, C_FILT_2, C_FILT_3, C_FILT_4, C_FILT_5, C_FILT_E_1, C_FILT_E_2: 0.1uF, Capacitor_SMD:C_0201_0603Metric, symbol Device:C
- added J_CLAMP: Screw_Terminal_01x10, TerminalBlock:TerminalBlock_MaiXu_MX126-5.0-10P_1x10_P5.00mm, symbol Connector:Screw_Terminal_01x10
- added R_DIV1_1, R_DIV1_2, R_DIV1_3, R_DIV1_4, R_DIV1_5: 10k, Resistor_SMD:R_0201_0603Metric, symbol Device:R
- added R_DIV2_1, R_DIV2_2, R_DIV2_3, R_DIV2_4, R_DIV2_5: 20k, Resistor_SMD:R_0201_0603Metric, symbol Device:R
- added R_FILT_1, R_FILT_2, R_FILT_3, R_FILT_4, R_FILT_5, R_SER_1, R_SER_2, R_SER_3, R_SER_4, R_SER_5: 1k, Resistor_SMD:R_0201_0603Metric, symbol Device:R
- added U2, U5: MCP6004, Package_SO:SOIC-14_3.9x8.7mm_P1.27mm, symbol Amplifier_Operational:MCP6004
Connections:
- new net: R_DIV1_5.2, R_SER_5.2
- new net: R_DIV1_3.1, R_DIV2_3.1, R_FILT_3.1
- new net: R_DIV1_4.1, R_DIV2_4.1, R_FILT_4.1
- new net: C_FILT_4.1, R_FILT_4.2, U2.12 (+)
- new net: R_DIV1_1.2, R_SER_1.2
- new net: R_DIV1_5.1, R_DIV2_5.1, R_FILT_5.1
- new net: C_FILT_1.1, R_FILT_1.2, U2.3 (+)
- new net: R_DIV1_1.1, R_DIV2_1.1, R_FILT_1.1
- new net: C_FILT_2.1, R_FILT_2.2, U2.5 (+)
- new net: R_DIV1_3.2, R_SER_3.2
- new net: R_DIV1_4.2, R_SER_4.2
- new net: C_FILT_5.1, R_FILT_5.2, U5.12 (+)
- new net: R_DIV1_2.1, R_DIV2_2.1, R_FILT_2.1
- new net: R_DIV1_2.2, R_SER_2.2
- new net: C_FILT_3.1, R_FILT_3.2, U2.10 (+)
- new net +3V3: C_FILT_E_1.1, C_FILT_E_2.1, U2.4 (V+), U5.4 (V+)
- new net ADC_CH0: U2.1, U2.2 (-)
- new net ADC_CH1: U2.6 (-), U2.7
- new net ADC_CH2: U2.8, U2.9 (-)
- new net ADC_CH3: U2.13 (-), U2.14
- new net ADC_CH4: U5.13 (-), U5.14
- new net CLAMP1_SIG: J_CLAMP.1 (Pin_1), R_SER_1.1
- new net CLAMP2_SIG: J_CLAMP.3 (Pin_3), R_SER_2.1
- new net CLAMP3_SIG: J_CLAMP.5 (Pin_5), R_SER_3.1
- new net CLAMP4_SIG: J_CLAMP.7 (Pin_7), R_SER_4.1
- new net CLAMP5_SIG: J_CLAMP.9 (Pin_9)
- new net CLAMP5__SIG: R_SER_5.1
- new net GND: C_FILT_1.2, C_FILT_2.2, C_FILT_3.2, C_FILT_4.2, C_FILT_5.2, C_FILT_E_1.2, C_FILT_E_2.2, J_CLAMP.10 (Pin_10), J_CLAMP.2 (Pin_2), J_CLAMP.4 (Pin_4), J_CLAMP.6 (Pin_6), J_CLAMP.8 (Pin_8), R_DIV2_1.2, R_DIV2_2.2, R_DIV2_3.2, R_DIV2_4.2, R_DIV2_5.2, U2.11 (V-), U5.11 (V-)
Other:
- company: (none) -> Don McGarry
