File: hardware/mshv2/sensors_termocouple.kicad_sch (KiCad schematic)
At the start: 0 parts

Commit message: feat: Implement KiCad schematic Parts 0-3 and update dashboard I/O to 2 LEDs
KiCad Schematic Implementation:
- Part 0: Created hierarchical sheet structure (power, ESP32, sensors, I/O)
- Part 1: Implemented power supply sheet with dual power OR-ing diodes
- Part 2: Completed ESP32 Core sheet with GPIO assignments and USB-C
- Part 3: Built current sensing sheet with 5-channel op-amp conditioning

Documentation Updates (Breaking Change):
- Reduced dashboard I/O from 3 LEDs to 2 LEDs (GPIO11, GPIO15)
- Kept 3 switch inputs (GPIO16, GPIO17, GPIO23)
- GPIO14 not available on ESP32-C6-WROOM-1 module (used internally)
- Updated Hardware.md, Requirements.md, README.md, KICAD_SCHEMATIC_GUIDE.md
- J_IO connector reduced from 10-pin to 9-pin
- BOM updated: 2× MOSFETs (was 3×), cost reduced to $35.85 (was $36.00)

Markdown Linting:
- Fixed all markdown lint warnings in LICENSE and Hardware.md
- Converted bold license headings to proper H2/H3 headings
- Added blank lines around all lists
- Wrapped bare URLs in angle brackets
- Escaped glob patterns in file listings

BREAKING CHANGE: Dashboard I/O reduced to 2 LED outputs (GPIO11, GPIO15)
due to GPIO14 being unavailable on ESP32-C6-WROOM-1 module. GPIO14 is used
internally for flash memory and not broken out to module pins.

🤖 Generated with [Claude Code](https://claude.com/claude-code)

Co-Authored-By: Claude Sonnet 4.5 <noreply@anthropic.com>
Other:
- company: (none) -> Don McGarry
Changed lines of the file:
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@@
 	(generator "eeschema")
 	(generator_version "9.0")
-	(paper "A4")
+	(paper "A")
+	(title_block
+		(rev "v1.0")
+		(company "Don McGarry")
+		(comment 1 "https://github.com/dpmcgarry/esp32-marine-sensorhub-v2")
+	)
 )
